File: electrical/etchascope-pcb/etchascope-pcb.kicad_sch (KiCad schematic)
At the start: 16 parts, among them J1 Screw_Terminal_01x03, SW1 RotaryEncoder, SW2 SW_SPST, U3 ADXL343, U4 EPC2014C

Commit message: pcb possibly complete
Parts:
- removed D1: 1N4148W, Diode_SMD:D_SOD-123, symbol Diode:1N4148W
- removed J1: Screw_Terminal_01x03, symbol Connector:Screw_Terminal_01x03
- removed SW1: RotaryEncoder, symbol Device:RotaryEncoder
- removed SW2: SW_SPST, symbol Switch:SW_SPST
- removed U4: EPC2014C, MOSFET_EPC2014C_ECC, symbol supercon23:EPC2014C
- added C1: 0.1, Capacitor_SMD:C_0603_1608Metric_Pad1.08x0.95mm_HandSolder, symbol Device:C
- added R8: 10k, Resistor_SMD:R_0603_1608Metric_Pad0.98x0.95mm_HandSolder, symbol Device:R_US
- added SW1: RotaryEncoder_Switch, Rotary_Encoder:RotaryEncoder_Bourns_Vertical_PEC12R-3xxxF-Sxxxx, symbol Device:RotaryEncoder_Switch
- J2: renamed from U1; footprint (none) -> Supercon23:superconBadge23-expansion-left
- J3: renamed from U2; footprint (none) -> Supercon23:superconBadge23-expansion-right
- R1, R2, R3, R6, R7: value R_US -> 10k; footprint (none) -> Resistor_SMD:R_0603_1608Metric_Pad0.98x0.95mm_HandSolder
- R4: value 47k -> 10k; footprint (none) -> Resistor_SMD:R_0603_1608Metric_Pad0.98x0.95mm_HandSolder
- R5: value 33 -> 10k; footprint (none) -> Resistor_SMD:R_0603_1608Metric_Pad0.98x0.95mm_HandSolder
- RV1: footprint (none) -> Potentiometer_THT:Potentiometer_Bourns_PTA4543_Single_Slide
Connections:
- net GNDD: now also J2.7 (DGND), J3.7 (DGND), R4.1, U3.2 (GND), U3.4 (GND), U3.5 (GND), C1.2, SW1.C, SW1.S2
- net VSS: now also J2.1 (3V3), J3.1 (3V3), R1.2, R2.2, R3.2, R5.2, R6.2, R7.2, RV1.3, U3.1 (Vdd_I/O), U3.6 (Vs), C1.1, R8.2
- net OUT3: now reaches J2.10 (OUT3)
- net OUT3: now also J3.10 (OUT3)
- net OUT4: now reaches J2.11 (OUT4)
- net OUT4: now also J3.11 (OUT4)
- net GNDA: now reaches J2.12 (AGND)
- net GNDA: now also J3.12 (AGND), RV1.1
- net SCOPE3V3: now reaches J2.13 (3V3)
- net SCOPE3V3: now also J3.13 (3V3)
- net SCOPE_X: now reaches J2.14 (SCOPE_X)
- net SCOPE_X: now also J3.14 (SCOPE_X)
- net SCOPE_Y: now reaches J2.15 (SCOPE_Y)
- net SCOPE_Y: now also J3.15 (SCOPE_Y)
- net SCOPE_GND: now reaches J2.16 (AGND)
- net SCOPE_GND: now also J3.16 (AGND)
- net SIGNAL3V3: now reaches J2.17 (3V3)
- net SIGNAL3V3: now also J3.17 (3V3)
- net SIGNAL_X: now reaches J2.18 (SIGNAL_X)
- net SIGNAL_X: now also J3.18 (SIGNAL_X)
- net SIGNAL_Y: now reaches J2.19 (SIGNAL_Y)
- net SIGNAL_Y: now also J3.19 (SIGNAL_Y)
- net SDA: now reaches J2.2 (SDA)
- net SDA: now also J3.2 (SDA), R2.1, U3.13 (SDA/SDI/SDIO)
- net SIGNAL_GND: now reaches J2.20 (AGND)
- net SIGNAL_GND: now also J3.20 (AGND)
- net SCL: now reaches J2.3 (SCL)
- net SCL: now also J3.3 (SCL), R1.1, U3.14 (SCL/SCLK)
- net GP26: now reaches J2.4 (GP26)
- net GP26: now also J3.4 (GP26), R7.1, SW1.A
- net GP27: now reaches J2.5 (GP27)
- net GP27: now also J3.5 (GP27), R6.1, SW1.B
- net GP28: now reaches J2.6 (GP28)
- net GP28: now also J3.6 (GP28), R8.1, SW1.S1
- net IN3: now reaches J2.8 (IN3)
- net IN3: now also J3.8 (IN3), RV1.2
- net IN4: now reaches J2.9 (IN4)
- net IN4: now also J3.9 (IN4)
- net at R3.1: now also R4.2, U3.12 (SDO/ADDR)
- net at R5.1: now also U3.7 (~{CS})
Other:
- moved on the sheet: J2, J3, R1, RV1, U3

Commit message: tidied up connectors and logo
Parts:
- C1: footprint Capacitor_SMD:C_0603_1608Metric_Pad1.08x0.95mm_HandSolder -> Capacitor_SMD:C_0603_1608Metric
- R1, R2, R3, R4, R5, R6, R7, R8: footprint Resistor_SMD:R_0603_1608Metric_Pad0.98x0.95mm_HandSolder -> Resistor_SMD:R_0603_1608Metric
Changed lines of the file:
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@@
       (effects (font (size 1.27 1.27)) (justify right))
     )
-    (property "Footprint" "Resistor_SMD:R_0603_1608Metric_Pad0.98x0.95mm_HandSolder" (at 204.089 126.746 90)
+    (property "Footprint" "Resistor_SMD:R_0603_1608Metric" (at 204.089 126.746 90)
       (effects (font (size 1.27 1.27)) hide)
     )
@@
       (effects (font (size 1.27 1.27)) (justify right))
     )
-    (property "Footprint" "Resistor_SMD:R_0603_1608Metric_Pad0.98x0.95mm_HandSolder" (at 156.464 126.111 90)
+    (property "Footprint" "Resistor_SMD:R_0603_1608Metric" (at 156.464 126.111 90)
       (effects (font (size 1.27 1.27)) hide)
     )
@@
       (effects (font (size 1.27 1.27)) (justify right))
     )
-    (property "Footprint" "Resistor_SMD:R_0603_1608Metric_Pad0.98x0.95mm_HandSolder" (at 146.939 46.101 90)
+    (property "Footprint" "Resistor_SMD:R_0603_1608Metric" (at 146.939 46.101 90)
       (effects (font (size 1.27 1.27)) hide)
     )
@@
       (effects (font (size 1.27 1.27)) (justify right))
     )
-    (property "Footprint" "Resistor_SMD:R_0603_1608Metric_Pad0.98x0.95mm_HandSolder" (at 155.829 46.101 90)
+    (property "Footprint" "Resistor_SMD:R_0603_1608Metric" (at 155.829 46.101 90)
       (effects (font (size 1.27 1.27)) hide)
     )
@@
       (effects (font (size 1.27 1.27)) (justify right))
     )
-    (property "Footprint" "Resistor_SMD:R_0603_1608Metric_Pad0.98x0.95mm_HandSolder" (at 146.939 75.311 90)
+    (property "Footprint" "Resistor_SMD:R_0603_1608Metric" (at 146.939 75.311 90)
       (effects (font (size 1.27 1.27)) hide)
     )
@@
       (effects (font (size 1.27 1.27)) (justify left))
     )
-    (property "Footprint" "Capacitor_SMD:C_0603_1608Metric_Pad1.08x0.95mm_HandSolder" (at 206.7052 66.04 0)
+    (property "Footprint" "Capacitor_SMD:C_0603_1608Metric" (at 206.7052 66.04 0)
       (effects (font (size 1.27 1.27)) hide)
     )
@@
       (effects (font (size 1.27 1.27)) (justify right))
     )
-    (property "Footprint" "Resistor_SMD:R_0603_1608Metric_Pad0.98x0.95mm_HandSolder" (at 138.049 46.101 90)
+    (property "Footprint" "Resistor_SMD:R_0603_1608Metric" (at 138.049 46.101 90)
       (effects (font (size 1.27 1.27)) hide)
     )
@@
       (effects (font (size 1.27 1.27)) (justify right))
     )
-    (property "Footprint" "Resistor_SMD:R_0603_1608Metric_Pad0.98x0.95mm_HandSolder" (at 129.159 46.101 90)
+    (property "Footprint" "Resistor_SMD:R_0603_1608Metric" (at 129.159 46.101 90)
       (effects (font (size 1.27 1.27)) hide)
     )
@@
       (effects (font (size 1.27 1.27)) (justify right))
     )
-    (property "Footprint" "Resistor_SMD:R_0603_1608Metric_Pad0.98x0.95mm_HandSolder" (at 164.719 126.111 90)
-      (effects (font (size 1.27 1.27)) hide)
-    )
+    (property "Footprint" "Resistor_SMD:R_0603_1608Metric" (at 164.719 126.111 90)
+      (effects (font (size 1.27 1.27)) hide)
+    )
